Commit message: Update robot_core.xacro

File: description/robot_core.xacro (robot description, xacro)
@@ -42,4 +42,7 @@
      </xacro:inertial_box>
    </link>
+   <gazebo reference="chassis">
+      <material>Gazebo/White</material>
+   </gazebo>
   <!-- LEFT WHEEL-->
    <joint name="left_wheel_joint" type="continuous">
@@ -65,4 +68,7 @@
      </xacro:inertial_cylinder>
     </link>
+    <gazebo reference="left_wheel">
+      <material>Gazebo/Blue</material>
+    </gazebo>
     <!-- RIGHT WHEEL -->
   <joint name="right_wheel_joint" type="continuous">
@@ -88,4 +94,7 @@
     </xacro:inertial_sphere>
   </link>
+   <gazebo reference="right_wheel">
+      <material>Gazebo/Blue</material>
+   </gazebo>
 <!-- CASTER WHEEL -->
   <joint name="caster_wheel_joint" type="fixed">
@@ -107,3 +116,8 @@
     </collision>
   </link>
+   <gazebo reference="caster_wheel">
+      <material>Gazebo/Black</material>
+      <mu1 value="0.001"/>
+      <mu2 value="0.001"/>
+   </gazebo>
 </robot>
